File: CM4_HighSpeed.kicad_sch (KiCad schematic)
At the start: 10 parts, among them J15 Conn_01x22_Female, J16 Conn_01x22_Female, J4 Conn_01x22_Female, J5 Conn_01x22_Female, J6 THD-02-R, U12 RT9742SNGV

Commit message: Add files via upload
Parts:
- removed J15, J16, J4, J5: Conn_01x22_Female, CM4IO:Hirose_FH12-22S-0.5SH_1x22-1MP_P0.50mm_Horizontal, symbol Connector:Conn_01x22_Female
Connections:
- net GND: no longer Module1.155 (GND)
- net CAM0_C_N: no longer names the net of Module1.140 (CAM0_C_N)
- net CAM0_C_P: no longer names the net of Module1.142 (CAM0_C_P)
- net CAM0_D0_N: no longer names the net of Module1.128 (CAM0_D0_N)
- net CAM0_D0_P: no longer names the net of Module1.130 (CAM0_D0_P)
- net CAM0_D1_N: no longer names the net of Module1.134 (CAM0_D1_N)
- net CAM0_D1_P: no longer names the net of Module1.136 (CAM0_D1_P)
- net CAM1_C_N: no longer names the net of Module1.127 (CAM1_C_N)
- net CAM1_C_P: no longer names the net of Module1.129 (CAM1_C_P)
- net CAM1_D0_N: no longer names the net of Module1.115 (CAM1_D0_N)
- net CAM1_D0_P: no longer names the net of Module1.117 (CAM1_D0_P)
- net CAM1_D1_N: no longer names the net of Module1.121 (CAM1_D1_N)
- net CAM1_D1_P: no longer names the net of Module1.123 (CAM1_D1_P)
- net CAM1_D2_N: no longer names the net of Module1.133 (CAM1_D2_N)
- net CAM1_D2_P: no longer names the net of Module1.135 (CAM1_D2_P)
- net CAM1_D3_N: no longer names the net of Module1.139 (CAM1_D3_N)
- net DSI0_C_N: no longer names the net of Module1.169 (DSI0_C_N)
- net DSI0_C_P: no longer names the net of Module1.171 (DSI0_C_P)
- net DSI0_D0_N: no longer names the net of Module1.157 (DSI0_D0_N)
- net DSI0_D0_P: no longer names the net of Module1.159 (DSI0_D0_P)
- net DSI0_D1_N: no longer names the net of Module1.163 (DSI0_D1_N)
- net DSI0_D1_P: no longer names the net of Module1.165 (DSI0_D1_P)
- net DSI1_C_N: no longer names the net of Module1.187 (DSI1_C_N)
- net DSI1_C_P: no longer names the net of Module1.189 (DSI1_C_P)
- net DSI1_D0_N: no longer names the net of Module1.175 (DSI1_D0_N)
- net DSI1_D0_P: no longer names the net of Module1.177 (DSI1_D0_P)
- net DSI1_D1_N: no longer names the net of Module1.181 (DSI1_D1_N)
- net DSI1_D1_P: no longer names the net of Module1.183 (DSI1_D1_P)
- net DSI1_D2_N: no longer names the net of Module1.193 (DSI1_D2_N)
- net DSI1_D2_P: no longer names the net of Module1.195 (DSI1_D2_P)
- net DSI1_D3_N: no longer names the net of Module1.194 (DSI1_D3_N)
- net DSI1_D3_P: no longer names the net of Module1.196 (DSI1_D3_P)
- no-connect marks 49 -> 51
Other:
- note removed: "Camera Connectors"
- note removed: "Display Connectors"
